Commit message: added mesh arg to ir_marker macro

File: urdf/sensors.urdf.xacro (robot description, xacro)
@@ -22,9 +22,8 @@
   </xacro:macro>
   <!-- Smocap Infrared Marker -->
-  <xacro:macro name="cs_smocap_ir_marker" params="*origin">
+  <xacro:macro name="cs_smocap_ir_marker" params="mesh *origin">
     <xacro:arg name="root_link" default="irm_link"/>
-    <xacro:arg name="mesh" default="ir_marker.dae"/>
     <xacro:include filename="$(find smocap)/urdf/ir_marker.urdf.xacro" />
-    <xacro:ir_marker root_link="$(arg root_link)" mesh="$(arg mesh)"/>
+    <xacro:ir_marker root_link="$(arg root_link)" mesh="${mesh}"/>
     <xacro:property name="irm_z" value="0.06" />
     <joint name="irm_joint" type="fixed">

Commit message: added 2D laser

File: urdf/sensors.urdf.xacro (robot description, xacro)
@@ -4,5 +4,5 @@
   <!-- Camera -->
   <xacro:macro name="cs_camera_eachine" params="*origin">
-    <link name="camera_link">
+    <link name="camera1_link">
     <visual>
       <xacro:if value="${high_definition_camera_visual}">
@@ -10,13 +10,20 @@
         <geometry><mesh scale="1. 1. 1." filename="package://common_robots/meshes/eachine_camera.dae"/></geometry>
       </xacro:if>
-      <xacro:unless value="${high_definition_wheel_visual}">
+      <xacro:unless value="${high_definition_camera_visual}">
 	<geometry><cylinder radius="0.0025" length="0.01"/></geometry><origin xyz="0 0 0" rpy="0 ${pi/2} 0"/>
       </xacro:unless>
     </visual>
   </link>
-  <joint name="camera_joint" type="fixed">
+  <joint name="camera1_joint" type="fixed">
     <xacro:insert_block name="origin"/>
     <parent link="base_link" />
-    <child link="camera_link" />
+    <child link="camera1_link" />
+  </joint>
+  <link name="camera1_optical_frame">
+  </link>
+  <joint name="camera1_optical_frame_joint" type="fixed">
+    <origin rpy="${-pi/2} 0.0 ${-pi/2}" xyz="0.0 0.0 0.0"/>
+    <parent link="camera1_link"/>
+    <child link="camera1_optical_frame"/>
   </joint>
   </xacro:macro>
@@ -33,3 +40,17 @@
     </joint>
   </xacro:macro>
+  <!-- Hokuyo 2D lidar -->
+  <xacro:macro name="cs_hokuyo" params="*origin">
+    <link name="hokuyo_link">
+      <visual>
+	<origin xyz="0 0 0" rpy="0 0 ${pi/2}"/>
+        <geometry><mesh scale="1. 1. 1." filename="package://common_robots/meshes/hokuyo.dae"/></geometry>
+      </visual>
+    </link>
+    <joint name="hokuyo_joint" type="fixed">
+      <xacro:insert_block name="origin"/>
+      <parent link="chassis_link"/>
+      <child link="hokuyo_link" />
+    </joint>
+  </xacro:macro>
 </robot>

Commit message: improving camera

File: urdf/sensors.urdf.xacro (robot description, xacro)
@@ -3,27 +3,27 @@
   <!-- Sensors -->
   <!-- Camera -->
-  <xacro:macro name="cs_camera_eachine" params="*origin">
-    <link name="camera1_link">
+  <xacro:macro name="cs_camera_eachine" params="cam_name origin_ref_frame *origin">
+    <link name="${cam_name}_link">
     <visual>
-      <xacro:if value="${high_definition_camera_visual}">
+      <xacro:if value="${cam_hd_visual}">
 	<origin xyz="0 0 0" rpy="0 0 ${pi/2}"/>
         <geometry><mesh scale="1. 1. 1." filename="package://common_robots/meshes/eachine_camera.dae"/></geometry>
       </xacro:if>
-      <xacro:unless value="${high_definition_camera_visual}">
+      <xacro:unless value="${cam_hd_visual}">
 	<geometry><cylinder radius="0.0025" length="0.01"/></geometry><origin xyz="0 0 0" rpy="0 ${pi/2} 0"/>
       </xacro:unless>
     </visual>
   </link>
-  <joint name="camera1_joint" type="fixed">
+  <joint name="${cam_name}_joint" type="fixed">
     <xacro:insert_block name="origin"/>
-    <parent link="base_link" />
-    <child link="camera1_link" />
+    <parent link="${origin_ref_frame}" />
+    <child link="${cam_name}_link" />
   </joint>
-  <link name="camera1_optical_frame">
+  <link name="${cam_name}_optical_frame">
   </link>
-  <joint name="camera1_optical_frame_joint" type="fixed">
+  <joint name="${cam_name}_optical_frame_joint" type="fixed">
     <origin rpy="${-pi/2} 0.0 ${-pi/2}" xyz="0.0 0.0 0.0"/>
-    <parent link="camera1_link"/>
-    <child link="camera1_optical_frame"/>
+    <parent link="${cam_name}_link"/>
+    <child link="${cam_name}_optical_frame"/>
   </joint>
   </xacro:macro>

Commit message: adding lidar

File: urdf/sensors.urdf.xacro (robot description, xacro)
@@ -54,3 +54,25 @@
     </joint>
   </xacro:macro>
+  <!-- Rplidar 2D lidar -->
+  <!-- TODO: finish that, use correct DAE and link names -->
+  <xacro:macro name="cs_rplidar" params="*origin">
+    <link name="hokuyo_link">
+      <visual>
+	<origin xyz="0 0 0" rpy="0 0 ${pi/2}"/>
+        <geometry><mesh scale="1. 1. 1." filename="package://common_robots/meshes/hokuyo.dae"/></geometry>
+      </visual>
+    </link>
+    <joint name="hokuyo_joint" type="fixed">
+      <xacro:insert_block name="origin"/>
+      <parent link="chassis_link"/>
+      <child link="hokuyo_link" />
+    </joint>
+  </xacro:macro>
+  <!-- Velodyne VLP16 lidar -->
+  <xacro:macro name="cs_vlp16" params="*origin">
+    <xacro:include filename="$(find velodyne_description)/urdf/VLP-16.urdf.xacro"/>
+    <VLP-16 parent="base_link" name="velodyne" topic="/velodyne_points" hz="10" samples="1024" gpu="false" lasers="16" max_range="100">
+      <xacro:insert_block name="origin"/>
+    </VLP-16>
+  </xacro:macro>
 </robot>
